File: Hardware/RaspberryPi_I2C_Isolator/RaspberryPi_I2C_Isolator.kicad_sch (KiCad schematic)
At the start: 25 parts, among them J1 Raspberry_Pi_2_3, J2 Conn_01x04_Male, J3 Conn_01x04_Male, J4 Conn_01x02_Male, U1 B0505LS-1WR3, U2 AMS1117-3.3, U3 ADuM1250ARZ, U4 ADS1115IDGS

Commit message: Edited the LED block title to "Status LED"
Other:
- note added: "Status LED"
Changed lines of the file:
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@@
     (effects (font (size 1.6 1.6)) (justify left bottom))
   )
-  (text "ADS1115 16-bit ADC" (at 15.24 160.02 0)
+  (text "Status LED" (at 15.24 160.02 0)
     (effects (font (size 2.54 2.54) (thickness 0.508) bold) (justify left bottom))
   )
